File: Hardware/RAFTv1.0/RAFT_DuckLink_NA.sch (EAGLE design)
At the start: 77 parts, among them J1 132134-15, J2 132134-15, U1 PE4259, U2 MAX2771ETI+, U3 SX1276, U4 PE4259, U5 PE4259, U6 PE4259

Commit message: finalized universal LoRa schematic. started power schematic. renamed schematics
Parts:
- removed C1, C2, C3, C61, C62, C63, C64, C69, C72, C74: (no value), rcl:C-USC0805
- removed C46, C47, C48, C49, C50: 100nF, rcl:C-USC0805
- removed C51, C52: 15pF, rcl:C-USC0805
- removed C53, C54, C66, C67, C75, C76: 47pF, rcl:C-USC0805
- removed C55: 10nF, rcl:C-USC0805
- removed C56: 47nF, rcl:C-USC0805
- removed C57: 8.2pF, rcl:C-USC0805
- removed C58: 22pF, rcl:C-USC0805
- removed C59, C70, C71: 6.8pF, rcl:C-USC0805
- removed C60: 3.3nH, rcl:C-USC0805
- removed C65: 3.3pF, rcl:C-USC0805
- removed C68, C77: 4.7pF, rcl:C-USC0805
- removed C73: 2.7nH, rcl:C-USC0805
- removed J1: 132134-15, 132134-15:132134-15
- removed L15: 33nH, rcl:L-USL3225M
- removed L16: 1.5nH, rcl:L-USL3225M
- removed L17: 82nH, rcl:L-USL3225M
- removed L18, L19: 5.6nH, rcl:L-USL3225M
- removed L20: 0H, rcl:L-USL3225M
- removed L21: (no value), rcl:L-USL3225M
- removed L22, L26: 15nH, rcl:L-USL3225M
- removed L23: 12nH, rcl:L-USL3225M
- removed L24: 0R, rcl:L-USL3225M
- removed L25: 18nH, rcl:L-USL3225M
- removed Q1: (no value), special:XTAL/S
- removed R2, R3, R4: 0R, rcl:R-US_R0805
- removed U3: SX1276, SX1276:SX1276
- removed U4, U5: PE4259, PE4259:PE4259
- added C10, C11: 15pF, rcl:C-USC0805
- added C12, C13, C25, C26, C80, C81: 47pF, rcl:C-USC0805
- added C14: 10nF, rcl:C-USC0805
- added C15: 47nF, rcl:C-USC0805
- added C16: 8.2pF, rcl:C-USC0805
- added C17: 22pF, rcl:C-USC0805
- added C18, C28, C29: 6.8pF, rcl:C-USC0805
- added C19: 3.3nH, rcl:C-USC0805
- added C24: 3.3pF, rcl:C-USC0805
- added C27, C82: 4.7pF, rcl:C-USC0805
- added C31: 2.7nH, rcl:C-USC0805
- added C5, C6, C7, C8, C9: 100nF, rcl:C-USC0805
- added C79: (no value), rcl:C-USC0805
- added C83, C84, C85: 1nF, rcl:C-USC0805
- added J3: 132134-15, 132134-15:132134-15
- added L1: 33nH, rcl:L-USL3225M
- added L11: 18nH, rcl:L-USL3225M
- added L12, L8: 15nH, rcl:L-USL3225M
- added L2: 1.5nH, rcl:L-USL3225M
- added L3: 82nH, rcl:L-USL3225M
- added L4, L5: 5.6nH, rcl:L-USL3225M
- added L9: 12nH, rcl:L-USL3225M
- added Q3: (no value), special:XTAL/S
- added R5: 0R, rcl:R-US_R0805
- added U10, U8, U9: PE4259, PE4259:PE4259
- added U7: SX1276, SX1276:SX1276
- U1: value PE4259 -> ESP32-D0WD; device PE4259:PE4259 -> ESP32-D0WD:ESP32-D0WD
Connections:
- removed net N$1: J1.SIG, U5.RFC
- removed net N$2: U4.RFC, U5.RF2
- removed net N$3: U3.DIO5, U5.CTRL
- removed net N$34: R2.1, U3.XTB
- removed net N$35: C47.1, U3.VR_ANA
- removed net N$36: C51.1, Q1.1, R2.2
- removed net N$37: C49.1, U3.VR_DIG
- removed net N$38: C52.1, Q1.2, U3.XTA
- removed net N$39: C53.1, C54.1, C55.1, L15.1, L17.2, U3.VR_PA
- removed net N$4: U1.RFC, U5.RF1
- removed net N$40: C68.2, C77.1, L17.1, U3.RFO_LF
- removed net N$41: C57.2, C58.1, L15.2, L16.2
- removed net N$42: L16.1, U3.PA_BOOST
- removed net N$43: C58.2, L18.1
- removed net N$44: C59.2, C62.1, L18.2, L19.1
- removed net N$45: C60.2, C62.2, C63.2, L19.2, L20.1
- removed net N$46: C61.2, C63.1, L20.2, U4.RF1
- removed net N$47: C70.1, C73.1, L22.2, L23.1
- removed net N$48: C64.2, L21.1, U3.RFI_HF(GND)
- removed net N$49: C65.2, C66.1, L21.2
- removed net N$50: C66.2, R3.1
- removed net N$51: C67.1, R3.2
- removed net N$52: C67.2, U4.RF2
- removed net N$53: C77.2, L22.1
- removed net N$54: C71.1, C73.2, C74.1
- removed net N$55: L23.2, L24.1
- removed net N$56: C72.1, C74.2, L24.2, U1.RF2
- removed net N$57: L25.1, L26.1, U3.RFI_LF
- removed net N$58: C69.1, C75.1, L26.2
- removed net N$59: C75.2, R4.2
- removed net N$60: C76.1, R4.1
- removed net N$61: C76.2, U1.RF1
- removed net N$90: U1.CTRL, U3.RXTX/RF_MOD, U4.CTRL
- new net N$10: C8.1, U7.VR_DIG
- new net N$11: C10.1, Q3.1, R5.2
- new net N$12: C11.1, Q3.2, U7.XTA
- new net N$13: R5.1, U7.XTB
- new net N$14: C12.1, C13.1, C14.1, L1.1, L3.2, U7.VR_PA
- new net N$15: L2.1, U7.PA_BOOST
- new net N$16: C27.2, C82.1, L3.1, U7.RFO_LF
- new net N$17: C17.2, L4.1
- new net N$18: C18.2, L4.2, L5.1
- new net N$19: C19.2, L5.2, U9.RF1
- new net N$20: C80.2, C81.1
- new net N$21: C24.2, C25.1, U7.RFI_HF(GND)
- new net N$23: C25.2, C26.1
- new net N$33: C26.2, U9.RF2
- new net N$62: C16.2, C17.1, L1.2, L2.2
- new net N$63: C28.1, C31.1, L8.2, L9.1
- new net N$64: C29.1, C31.2, L9.2, U8.RF2
- new net N$67: L11.1, L12.1, U7.RFI_LF
- new net N$68: C79.1, C80.1, L12.2
- new net N$71: C81.2, U8.RF1
- new net N$72: C82.2, L8.1
- new net N$73: U7.RXTX/RF_MOD, U8.CTRL, U9.CTRL
- new net N$74: U10.RF1, U8.RFC
- new net N$75: U10.RF2, U9.RFC
- new net N$76: J3.SIG, U10.RFC
- new net N$77: U10.CTRL, U7.DIO5
- new net N$9: C6.1, U7.VR_ANA
- net GND: now also C10.2, C11.2, C12.2, C13.2, C14.2, C15.2, C16.1, C18.1, C19.1, C24.1, C27.1, C28.2, C29.2, C5.2, C6.2, C7.2, C79.2, C8.2, C83.2, C84.2, C85.2, C9.2, L11.2, U10.GND, U7.EXP, U7.GND, U7.RFO_HF(GND), U8.GND, U9.GND; no longer C1.2, C2.2, C3.2, C46.2, C47.2, C48.2, C49.2, C50.2, C51.2, C52.2, C53.2, C54.2, C55.2, C56.2, C57.1, C59.1, C60.1, C61.1, C64.1, C65.1, C68.1, C69.2, C70.2, C71.2, C72.2, L25.2, U1.GND, U3.EXP, U3.GND, U3.RFO_HF(GND), U4.GND, U5.GND
- net MISO: now also U7.MISO; no longer U3.MISO
- net MOSI: now also U7.MOSI; no longer U3.MOSI
- net SPI_CLK: now also U7.SCK; no longer U3.SCK
- net SX_CS: now also U7.NSS; no longer U3.NSS
- net VCC: now also C15.1, C5.1, C7.1, C83.1, C84.1, C85.1, C9.1, U10.!CTRL/!VDD, U7.VBAT_ANA, U7.VBAT_DIG, U7.VBAT_RF, U8.!CTRL/!VDD, U9.!CTRL/!VDD; no longer C1.1, C2.1, C3.1, C46.1, C48.1, C50.1, C56.1, U1.!CTRL/!VDD, U3.VBAT_ANA, U3.VBAT_DIG, U3.VBAT_RF, U4.!CTRL/!VDD, U5.!CTRL/!VDD
Other:
- note added: "1.5"
- note added: "SX1276 RFH NA ONLY"
- note removed: "1.2"
- note removed: "SX1276 RFH RFL - ref design"
